File: Keyboard/Keyboard.kicad_sch (KiCad schematic)
At the start: 253 parts, among them J1 TYPE-C-31-M-12, SW1 RotaryEncoder_Switch

Commit message: Add files via upload
Parts:
- removed D14, D30, D45, D59, D72, D73, D81, D82, D83: BAV16W, Diode_SMD:D_SOD-123, symbol Diode:BAV16W
- removed J1: TYPE-C-31-M-12, Keyboard:HRO_TYPE-C-31-M-12, symbol Keyboard:TYPE-C-31-M-12
- removed LED1, LED10, LED11, LED12, LED13, LED14, LED15, LED16, LED17, LED18, LED19, LED2, LED20, LED21, LED22, LED23, LED24, LED25, LED26, LED27, LED28, LED29, LED3, LED30, LED31, LED32, LED33, LED34, LED35, LED36, LED37, LED38, LED39, LED4, LED40, LED41, LED42, LED43, LED44, LED45, LED46, LED47, LED48, LED49, LED5, LED50, LED51, LED52, LED53, LED54, LED55, LED56, LED57, LED58, LED59, LED6, LED60, LED61, LED62, LED63, LED64, LED65, LED66, LED67, LED68, LED69, LED7, LED70, LED71, LED72, LED73, LED74, LED75, LED76, LED77, LED78, LED79, LED8, LED80, LED81, LED82, LED9: MX_SK6812MINI-E, PCM_marbastlib-mx:LED_MX_6028R, symbol PCM_marbastlib-mx:MX_SK6812MINI-E
- removed MX14, MX29, MX44, MX58, MX71, MX72, MX80, MX81, MX82: MX_SW_HS, PCM_marbastlib-mx:SW_MX_HS_CPG151101S11_1u, symbol PCM_marbastlib-mx:MX_SW_HS_CPG151101S11
- added A1: RaspberryPi_Pico, Keyboard:Raspberry PiPico, symbol MCU_Module:RaspberryPi_Pico
Connections:
- net Col 15 is gone; now on net Col 14: SW1.S2
- net +5V: now also A1.40 (VBUS)
- net Col 1: now also A1.1 (GPIO0)
- net Col 10: now also A1.15 (GPIO11)
- net Col 11: now also A1.14 (GPIO10)
- net Col 12: now also A1.12 (GPIO9); no longer MX70.1
- net Col 13: now also MX70.1, A1.19 (GPIO14); no longer MX57.1
- net Col 14: now also MX57.1, A1.10 (GPIO7)
- net Col 2: now also A1.2 (GPIO1)
- net Col 3: now also A1.4 (GPIO2)
- net Col 4: now also A1.5 (GPIO3); no longer MX76.1
- net Col 5: now also A1.6 (GPIO4)
- net Col 6: now also MX76.1, A1.7 (GPIO5)
- net Col 7: now also A1.21 (GPIO16)
- net Col 8: now also A1.22 (GPIO17)
- net Col 9: now also A1.16 (GPIO12)
- net GND: now also A1.13 (GND), A1.18 (GND), A1.23 (GND), A1.28 (GND), A1.3 (GND), A1.33 (AGND), A1.38 (GND), A1.8 (GND)
- net GPIO A: now also A1.26 (GPIO20)
- net GPIO B: now also A1.27 (GPIO21)
- net LED In: now also A1.20 (GPIO15)
- net Row 1: now also A1.29 (GPIO22)
- net Row 2: now also A1.25 (GPIO19)
- net Row 3: now also A1.24 (GPIO18)
- net Row 4: now also A1.11 (GPIO8)
- net Row 5: now also A1.17 (GPIO13); no longer D74.1 (K), D75.1 (K), D76.1 (K), D77.1 (K), D78.1 (K), D79.1 (K), D80.1 (K)
- new net Row 6: A1.9 (GPIO6), D74.1 (K), D75.1 (K), D76.1 (K), D77.1 (K), D78.1 (K), D79.1 (K), D80.1 (K)
- no-connect marks 0 -> 8
Other:
- added sheet Leds (Leds.kicad_sch)
- moved on the sheet: D15, D58, D71, D77, MX57, MX70, MX76, SW1

Commit message: Add files via upload
Parts:
- removed D80: BAV16W, Diode_SMD:D_SOD-123, symbol Diode:BAV16W
- removed MX79: MX_SW_HS, PCM_marbastlib-mx:SW_MX_HS_CPG151101S11_1u, symbol PCM_marbastlib-mx:MX_SW_HS_CPG151101S11
Connections:
- net Col 10: now also A1.11 (GPIO8); no longer A1.15 (GPIO11)
- net Col 11: now also A1.12 (GPIO9); no longer A1.14 (GPIO10)
- net Col 12: now also A1.10 (GPIO7); no longer A1.12 (GPIO9)
- net Col 13: now also A1.15 (GPIO11); no longer A1.19 (GPIO14)
- net Col 14: now also A1.17 (GPIO13); no longer A1.10 (GPIO7)
- net Col 9: now also A1.19 (GPIO14); no longer A1.16 (GPIO12)
- net Row 2: now also A1.24 (GPIO18); no longer A1.25 (GPIO19)
- net Row 3: now also A1.25 (GPIO19); no longer A1.24 (GPIO18)
- net Row 4: now also A1.16 (GPIO12); no longer A1.11 (GPIO8)
- net Row 5: now also A1.14 (GPIO10); no longer A1.17 (GPIO13)
