File: Keyboard/Leds.kicad_sch (KiCad schematic)
At the start: 146 parts

Commit message: Add files via upload
Parts:
- added C74: 1000uF, Capacitor_SMD:C_0805_2012Metric, symbol Device:C
- added R1: 470, Capacitor_SMD:C_0805_2012Metric, symbol Device:R
Connections:
- net +5V: now also C74.2
- net GND: now also C74.1
- net LED In: now also R1.1; no longer LED1.3 (DIN)
- new net: LED1.3 (DIN), R1.2
Other:
- note added: "Bulk Cap and Data Resistor"
Changed lines of the file:
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@@
 	(generator_version "9.0")
 	(paper "A3")
+	(text "Bulk Cap and Data Resistor\n"
+		(exclude_from_sim no)
+		(at 37.338 25.908 0)
+		(effects
+			(font
+				(size 1.27 1.27)
+			)
+		)
+	)
 	(junction
 		(at 248.92 107.95)
@@
 	)
 	(junction
+		(at 76.2 35.56)
+		(diameter 0)
+		(color 0 0 0 0)
+	)
+	(junction
 		(at 76.2 31.75)
 		(diameter 0)
@@
 	)
 	(junction
+		(at 76.2 43.18)
+		(diameter 0)
+		(color 0 0 0 0)
+	)
+	(junction
 		(at 238.76 92.71)
 		(diameter 0)
@@
 	(wire
 		(pts
+			(xy 44.45 35.56) (xy 76.2 35.56)
+		)
+		(stroke
+			(width 0)
+			(type default)
+		)
+	)
+	(wire
+		(pts
 			(xy 309.88 107.95) (xy 299.72 107.95)
 		)
@@
 	(wire
 		(pts
+			(xy 44.45 43.18) (xy 76.2 43.18)
+		)
+		(stroke
+			(width 0)
+			(type default)
+		)
+	)
+	(wire
+		(pts
 			(xy 208.28 46.99) (xy 218.44 46.99)
 		)
@@
 	(global_label "LED In"
 		(shape input)
-		(at 64.77 39.37 180)
+		(at 57.15 39.37 180)
 		(fields_autoplaced yes)
 		(effects
@@
 		)
 		(property "Intersheetrefs" "${INTERSHEET_REFS}"
-			(at 55.6163 39.37 0)
+			(at 47.9963 39.37 0)
 			(effects
 				(font
@@
 	)
 	(symbol
+		(lib_id "Device:R")
+		(at 60.96 39.37 90)
+		(unit 1)
+		(exclude_from_sim no)
+		(in_bom yes)
+		(on_board yes)
+		(dnp no)
+		(fields_autoplaced yes)
+		(property "Reference" "R1"
+			(at 60.96 33.02 90)
+			(effects
+				(font
+					(size 1.27 1.27)
+				)
+			)
+		)
+		(property "Value" "470"
+			(at 60.96 35.56 90)
+			(effects
+				(font
+					(size 1.27 1.27)
+				)
+			)
+		)
+		(property "Footprint" "Capacitor_SMD:C_0805_2012Metric"
+			(at 60.96 41.148 90)
+			(effects
+				(font
+					(size 1.27 1.27)
+				)
+				(hide yes)
+			)
+		)
+		(property "Datasheet" "~"
+			(at 60.96 39.37 0)
+			(effects
+				(font
+					(size 1.27 1.27)
+				)
+				(hide yes)
+			)
+		)
+		(property "Description" "Resistor"
+			(at 60.96 39.37 0)
+			(effects
+				(font
+					(size 1.27 1.27)
+				)
+				(hide yes)
+			)
+		)
+		(pin "2"
+		)
+		(pin "1"
+		)
+		(instances
+			(project ""
+				(path "/1adb6431-6ef0-4791-a9b7-77cd24f5e50e/8000d41a-6d92-4955-bded-3e4555e4e3bb"
+					(reference "R1")
+					(unit 1)
+				)
+			)
+		)
+	)
+	(symbol
 		(lib_id "PCM_marbastlib-various:SK6812MINI-E")
 		(at 309.88 39.37 0)
@@
 					(unit 1)
 				)
+			)
+		)
+	)
+	(symbol
+		(lib_id "Device:C")
+		(at 44.45 39.37 180)
+		(unit 1)
+		(exclude_from_sim no)
+		(in_bom yes)
+		(on_board yes)
+		(dnp no)
+		(property "Reference" "C74"
+			(at 36.322 37.846 0)
+			(effects
+				(font
+					(size 1.27 1.27)
+				)
+				(justify right)
+			)
+		)
+		(property "Value" "1000uF"
+			(at 35.56 40.64 0)
+			(effects
+				(font
+					(size 1.27 1.27)
+				)
+				(justify right)
+			)
+		)
+		(property "Footprint" "Capacitor_SMD:C_0805_2012Metric"
+			(at 43.4848 35.56 0)
+			(effects
+				(font
+					(size 1.27 1.27)
+				)
+				(hide yes)
+			)
+		)
+		(property "Datasheet" "~"
+			(at 44.45 39.37 0)
+			(effects
+				(font
+					(size 1.27 1.27)
+				)
+				(hide yes)
+			)
+		)
+		(property "Description" "Unpolarized capacitor"
+			(at 44.45 39.37 0)
+			(effects
+				(font
+					(size 1.27 1.27)
+				)
+				(hide yes)
+			)
+		)
+		(pin "2"
+		)
+		(pin "1"
+		)
+		(instances
+			(project "Keyboard"
+				(path "/1adb6431-6ef0-4791-a9b7-77cd24f5e50e/8000d41a-6d92-4955-bded-3e4555e4e3bb"
+					(reference "C74")
+					(unit 1)
+				)

Commit message: Add files via upload
Parts:
- removed C1: 100nF, Capacitor_SMD:C_0805_2012Metric, symbol Device:C
- removed LED1: SK6812MINI-E, PCM_marbastlib-mx:LED_MX_6028R, symbol PCM_marbastlib-various:SK6812MINI-E
Connections:
- net at R1.2: now also LED2.3 (DIN)
Changed lines of the file:
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@@
 	)
 	(junction
-		(at 76.2 35.56)
-		(diameter 0)
-		(color 0 0 0 0)
-	)
-	(junction
 		(at 76.2 31.75)
 		(diameter 0)
@@
 	)
 	(junction
-		(at 86.36 31.75)
-		(diameter 0)
-		(color 0 0 0 0)
-	)
-	(junction
 		(at 330.2 123.19)
 		(diameter 0)
@@
 	)
 	(junction
-		(at 76.2 43.18)
-		(diameter 0)
-		(color 0 0 0 0)
-	)
-	(junction
 		(at 238.76 92.71)
 		(diameter 0)
@@
 	(wire
 		(pts
-			(xy 64.77 39.37) (xy 78.74 39.37)
+			(xy 64.77 39.37) (xy 99.06 39.37)
 		)
 		(stroke
@@
 	(wire
 		(pts
-			(xy 86.36 31.75) (xy 96.52 31.75)
-		)
-		(stroke
-			(width 0)
-			(type default)
-		)
-	)
-	(wire
-		(pts
 			(xy 218.44 119.38) (xy 218.44 123.19)
 		)
@@
 	(wire
 		(pts
-			(xy 93.98 39.37) (xy 99.06 39.37)
-		)
-		(stroke
-			(width 0)
-			(type default)
-		)
-	)
-	(wire
-		(pts
 			(xy 299.72 35.56) (xy 299.72 31.75)
 		)
@@
 	(wire
 		(pts
-			(xy 76.2 31.75) (xy 86.36 31.75)
+			(xy 76.2 31.75) (xy 96.52 31.75)
 		)
 		(stroke
@@
 	(symbol
 		(lib_id "PCM_marbastlib-various:SK6812MINI-E")
-		(at 86.36 39.37 0)
-		(unit 1)
-		(exclude_from_sim no)
-		(in_bom yes)
-		(on_board yes)
-		(dnp no)
-		(fields_autoplaced yes)
-		(property "Reference" "LED1"
-			(at 100.33 32.9498 0)
-			(effects
-				(font
-					(size 1.27 1.27)
-				)
-			)
-		)
-		(property "Value" "SK6812MINI-E"
-			(at 100.33 35.4898 0)
-			(effects
-				(font
-					(size 1.27 1.27)
-				)
-			)
-		)
-		(property "Footprint" "PCM_marbastlib-mx:LED_MX_6028R"
-			(at 86.36 39.37 0)
-			(effects
-				(font
-					(size 1.27 1.27)
-				)
-				(hide yes)
-			)
-		)
-		(property "Datasheet" ""
-			(at 86.36 39.37 0)
-			(effects
-				(font
-					(size 1.27 1.27)
-				)
-				(hide yes)
-			)
-		)
-		(property "Description" "Reverse mount adressable LED (WS2812 protocol)"
-			(at 86.36 39.37 0)
-			(effects
-				(font
-					(size 1.27 1.27)
-				)
-				(hide yes)
-			)
-		)
-		(pin "3"
-		)
-		(pin "4"
-		)
-		(pin "2"
-		)
-		(pin "1"
-		)
-		(instances
-			(project ""
-				(path "/1adb6431-6ef0-4791-a9b7-77cd24f5e50e/8000d41a-6d92-4955-bded-3e4555e4e3bb"
-					(reference "LED1")
-					(unit 1)
-				)
-			)
-		)
-	)
-	(symbol
-		(lib_id "PCM_marbastlib-various:SK6812MINI-E")
 		(at 289.56 54.61 180)
 		(unit 1)
@@
 					(unit 1)
 				)
-			)
-		)
-	)
-	(symbol
-		(lib_id "Device:C")
-		(at 76.2 39.37 180)
-		(unit 1)
-		(exclude_from_sim no)
-		(in_bom yes)
-		(on_board yes)
-		(dnp no)
-		(fields_autoplaced yes)
-		(property "Reference" "C1"
-			(at 68.58 39.37 90)
-			(effects
-				(font
-					(size 1.27 1.27)
-				)
-			)
-		)
-		(property "Value" "100nF"
-			(at 71.12 39.37 90)
-			(effects
-				(font
-					(size 1.27 1.27)
-				)
-			)
-		)
-		(property "Footprint" "Capacitor_SMD:C_0805_2012Metric"
-			(at 75.2348 35.56 0)
-			(effects
-				(font
-					(size 1.27 1.27)
-				)
-				(hide yes)
-			)
-		)
-		(property "Datasheet" "~"
-			(at 76.2 39.37 0)
-			(effects
-				(font
-					(size 1.27 1.27)
-				)
-				(hide yes)
-			)
-		)
-		(property "Description" "Unpolarized capacitor"
-			(at 76.2 39.37 0)
-			(effects
-				(font
-					(size 1.27 1.27)
-				)
-				(hide yes)
-			)
-		)
-		(pin "2"
-		)
-		(pin "1"
-		)
-		(instances
-			(project ""
-				(path "/1adb6431-6ef0-4791-a9b7-77cd24f5e50e/8000d41a-6d92-4955-bded-3e4555e4e3bb"
-					(reference "C1")
-					(unit 1)
-				)
